File: CPU.sch (KiCad schematic (older format))
At the start: 25 parts, among them J1 10.0402_LCD_RGB_CON_WJQ, SW1 11.0101_SW-A03-08, U1 08.0001_F1C200S, Y1 07.0403_Crystal_24M_3225

Commit message: Removed TV. Added USB. Refactored.
Signed-off-by: Sebastian Basierski <sebastian@basierski.pl>
Parts:
- added TP1: TestPoint, TestPoint:TestPoint_Pad_1.0x1.0mm, symbol Connector:TestPoint
- C1, C11, C12, C2, C5: symbol 0WJQ:03.4004_C0603_10uF -> F1C200S_KIT-rescue:03.4004_C0603_10uF-0WJQ
- C10, C13, C14, C15, C3, C4, C6, C7, C8, C9: symbol 0WJQ:03.0009_C0402_100nF -> F1C200S_KIT-rescue:03.0009_C0402_100nF-0WJQ
- C16: symbol 0WJQ:03.0001_C0402_1uF -> F1C200S_KIT-rescue:03.0001_C0402_1uF-0WJQ
- C17, C18: symbol 0WJQ:03.0003_C0402_10pF -> F1C200S_KIT-rescue:03.0003_C0402_10pF-0WJQ
- J1: symbol 0WJQ:10.0402_LCD_RGB_CON_WJQ -> F1C200S_KIT-rescue:10.0402_LCD_RGB_CON_WJQ-0WJQ
- R1, R2: symbol 0WJQ:02.0026_R0402_2K_1% -> F1C200S_KIT-rescue:02.0026_R0402_2K_1%-0WJQ
- R3: symbol 0WJQ:02.0008_R0402_10K_1% -> F1C200S_KIT-rescue:02.0008_R0402_10K_1%-0WJQ
- SW1: symbol 0WJQ:11.0101_SW-A03-08 -> F1C200S_KIT-rescue:11.0101_SW-A03-08-0WJQ
- U1: symbol 0WJQ:08.0001_F1C200S -> F1C200S_KIT-rescue:08.0001_F1C200S-0WJQ
- Y1: symbol 0WJQ:07.0403_Crystal_24M_3225 -> F1C200S_KIT-rescue:07.0403_Crystal_24M_3225-0WJQ
Connections:
- net labels removed: FMINL, FMINR, HP_COM, HP_COMFB, HP_L, HP_R, LINL, LRADC0, MICIN, TV_IN0, TV_IN1, TV_OUT, TV_VCC, TV_VRN, TV_VRP, VRA1, VRA2
- wire segments 241 -> 217
- no-connect marks 2 -> 18
