File: Misc.sch (KiCad schematic (older format))
At the start: 23 parts, among them J2 10.0002_USB_Micro, J3 10.0001_Micro_SD_Card, J4 10.0201_PH2X15_2D54_V, J5 10.0002_USB_Micro, U4 09.0001_CP2104, U5 09.0303_GD5F1GQ4, U6 09.0302_W25Q128JVS

Commit message: Removed TV. Added USB. Refactored.
Signed-off-by: Sebastian Basierski <sebastian@basierski.pl>
Parts:
- removed C31: 03.4001_C0603_1uF, 0WJQ:C_0603_WJQ, symbol 0WJQ:03.4001_C0603_1uF
- removed C33: 03.4002_C0603_2.2uF, 0WJQ:C_0603_WJQ, symbol 0WJQ:03.4002_C0603_2.2uF
- removed C34: 03.0009_C0402_100nF, 0WJQ:C_0402_WJQ, symbol 0WJQ:03.0009_C0402_100nF
- removed D3, D4, D5: 07.0002_D_TVS_PESDNC2FD5VB, 0WJQ:DFN1006-2L, symbol 0WJQ:07.0002_D_TVS_PESDNC2FD5VB
- removed J2, J5: 10.0002_USB_Micro, 0WJQ:MicroUSB_5S_B_A01SB141B1-067, symbol 0WJQ:10.0002_USB_Micro
- removed R18: 02.0005_R0402_4K7_1%, 0WJQ:R_0402_WJQ, symbol 0WJQ:02.0005_R0402_4K7_1%
- removed R20: 02.0008_R0402_10K_1%, 0WJQ:R_0402_WJQ, symbol 0WJQ:02.0008_R0402_10K_1%
- removed U4: 09.0001_CP2104, Package_DFN_QFN:QFN-24-1EP_4x4mm_P0.5mm_EP2.6x2.6mm, symbol 0WJQ:09.0001_CP2104
- C36, C37: symbol 0WJQ:03.0009_C0402_100nF -> F1C200S_KIT-rescue:03.0009_C0402_100nF-0WJQ
- J3: symbol 0WJQ:10.0001_Micro_SD_Card -> F1C200S_KIT-rescue:10.0001_Micro_SD_Card-0WJQ
- J4: symbol 0WJQ:10.0201_PH2X15_2D54_V -> F1C200S_KIT-rescue:10.0201_PH2X15_2D54_V-0WJQ
- R13, R14, R15, R16, R17: symbol 0WJQ:02.0014_R0402_47K_1% -> F1C200S_KIT-rescue:02.0014_R0402_47K_1%-0WJQ
- R19: symbol 0WJQ:02.0008_R0402_10K_1% -> F1C200S_KIT-rescue:02.0008_R0402_10K_1%-0WJQ
- U5: symbol 0WJQ:09.0303_GD5F1GQ4 -> F1C200S_KIT-rescue:09.0303_GD5F1GQ4-0WJQ
- U6: symbol 0WJQ:09.0302_W25Q128JVS -> F1C200S_KIT-rescue:09.0302_W25Q128JVS-0WJQ
Connections:
- net labels removed: CP2104_RST, CPU_RXD, CPU_TXD, USB_D+, USB_D-, USB_ID, VBUS
- wire segments 131 -> 83
- no-connect marks 20 -> 5
Other:
- note removed: "Note: add tvs\n"
