File: Power.sch (KiCad schematic (older format))
At the start: 30 parts, among them U2 09.0103_XC6206, U3 09.0102_EA3036

Commit message: Removed TV. Added USB. Refactored.
Signed-off-by: Sebastian Basierski <sebastian@basierski.pl>
Parts:
- C19, C21, C22, C23, C27, C28, C29: symbol 0WJQ:03.4004_C0603_10uF -> F1C200S_KIT-rescue:03.4004_C0603_10uF-0WJQ
- C20, C24, C25, C26: symbol 0WJQ:03.0009_C0402_100nF -> F1C200S_KIT-rescue:03.0009_C0402_100nF-0WJQ
- C30: symbol 0WJQ:04.0002_CP1210_47uF -> F1C200S_KIT-rescue:04.0002_CP1210_47uF-0WJQ
- D1: symbol 0WJQ:07.0201_LED_Red_0603 -> F1C200S_KIT-rescue:07.0201_LED_Red_0603-0WJQ
- F1: symbol 0WJQ:07.0004_Fuse_0805_500mA -> F1C200S_KIT-rescue:07.0004_Fuse_0805_500mA-0WJQ
- H1, H2: symbol 0WJQ:MountingHole_Pad_M3 -> F1C200S_KIT-rescue:MountingHole_Pad_M3-0WJQ
- L1, L2, L3: symbol 0WJQ:06.0102_L2520_2.2uH -> F1C200S_KIT-rescue:06.0102_L2520_2.2uH-0WJQ
- R10: symbol 0WJQ:02.0024_R0402_470K_1% -> F1C200S_KIT-rescue:02.0024_R0402_470K_1%-0WJQ
- R11, R6, R7, R8: symbol 0WJQ:02.0023_R0402_150K_1% -> F1C200S_KIT-rescue:02.0023_R0402_150K_1%-0WJQ
- R4: symbol 0WJQ:02.0003_R0402_1K_1% -> F1C200S_KIT-rescue:02.0003_R0402_1K_1%-0WJQ
- R5: symbol 0WJQ:02.0001_R0402_0R_1% -> F1C200S_KIT-rescue:02.0001_R0402_0R_1%-0WJQ
- R9: symbol 0WJQ:02.0025_R0402_680K_1% -> F1C200S_KIT-rescue:02.0025_R0402_680K_1%-0WJQ
- U2: symbol 0WJQ:09.0103_XC6206P302MR -> F1C200S_KIT-rescue:09.0103_XC6206P302MR-0WJQ
- U3: symbol 0WJQ:09.0102_EA3036 -> F1C200S_KIT-rescue:09.0102_EA3036-0WJQ
